Commit message: added the two finger arm version

File: description_files/rover_arm_description/urdf/test_rover_arm.urdf.xacro (robot description, xacro)
@@ -1,4 +1,4 @@
 <?xml version="1.0"?>
-<robot xmlns:xacro="http://www.ros.org/wiki/xacro" name="test_rover_body">
+<robot xmlns:xacro="http://www.ros.org/wiki/xacro" name="test_rover_arm">
   <xacro:include filename="$(find rover_arm_description)/urdf/rover_arm.urdf.xacro" />
   <link name="base_link"/>

File: description_files/rover_arm_description/urdf/two_finger_arm.urdf.xacro (robot description, xacro)
@@ -1,5 +1,5 @@
 <?xml version="1.0"?>
-<robot xmlns:xacro="http://www.ros.org/wiki/xacro" name="rover_arm">
-  <xacro:macro name="rover_arm" params="parent prefix *origin">
+<robot xmlns:xacro="http://www.ros.org/wiki/xacro" name="rover_two_finger_arm">
+  <xacro:macro name="rover_two_finger_arm" params="parent prefix *origin">
   <!--
  __      __     _____  _____          ____  _      ______  _____
@@ -15,4 +15,6 @@
   <xacro:property name="j2_rotation_offset" value="${pi / 6} 0 0" />
   <xacro:property name="j3_rotation_offset" value="${pi - 0.4366117} 0 0" />
+  <xacro:property name="finger1_rotation_offset" value="0 0 ${pi / 2}" />
+  <xacro:property name="finger2_rotation_offset" value="${pi} 0 ${pi / 2}" />
   <!-- JOINT POSITIONS -->
   <xacro:property name="j1_joint_pos" value="0 0 0.024" />
@@ -21,10 +23,8 @@
   <xacro:property name="ee_base_joint_pos" value="-0.028 0 0.2715" />
   <xacro:property name="slider_joint_pos" value="0 0.11 0" />
-  <xacro:property name="finger1_joint_pos" value="-0.052384 0.134522 -0.016965" />
-  <xacro:property name="finger1_joint_rotation" value="0 ${-pi / 6} 0" />
-  <xacro:property name="finger2_joint_pos" value="0.011500 0.134522 0.053848" />
-  <xacro:property name="finger2_joint_rotation" value="0 ${pi / 2} 0" />
-  <xacro:property name="finger3_joint_pos" value="0.040884 0.134522 -0.036883" />
-  <xacro:property name="finger3_joint_rotation" value="0 ${pi * 7 / 6} 0" />
+  <xacro:property name="finger1_joint_pos" value="0.012017 0.156 -0.054914" />
+  <xacro:property name="finger1_joint_rotation" value="0 0 0" />
+  <xacro:property name="finger2_joint_pos" value="-0.012017 0.156 0.054914" />
+  <xacro:property name="finger2_joint_rotation" value="0 0 0" />
   <!-- COLORS -->
   <!-- links color -->
@@ -132,5 +132,5 @@
       <origin xyz="0 0.018007 0" rpy="0 0 0"/>
       <geometry>
-        <mesh filename="package://rover_arm_description/meshes/visual/end_effector_base.stl" scale="0.001 0.001 0.001"/>
+        <mesh filename="package://rover_arm_description/meshes/visual/two_finger_version/end_effector_base.stl" scale="0.001 0.001 0.001"/>
       </geometry>
       <material name="${prefix}links_color"/>
@@ -148,5 +148,5 @@
       <origin xyz="0 0 0" rpy="0 0 0"/>
       <geometry>
-        <mesh filename="package://rover_arm_description/meshes/visual/end_effector_slider.stl" scale="0.001 0.001 0.001"/>
+        <mesh filename="package://rover_arm_description/meshes/visual/two_finger_version/end_effector_slider.stl" scale="0.001 0.001 0.001"/>
       </geometry>
       <material name="${prefix}links_color"/>
@@ -157,7 +157,7 @@
   <link name="${prefix}ee_finger1">
     <visual>
-      <origin xyz="0 0 0" rpy="0 0 0"/>
-      <geometry>
-        <mesh filename="package://rover_arm_description/meshes/visual/end_effector_finger.stl" scale="0.001 0.001 0.001"/>
+      <origin xyz="0 0 0" rpy="${finger1_rotation_offset}"/>
+      <geometry>
+        <mesh filename="package://rover_arm_description/meshes/visual/two_finger_version/end_effector_finger.stl" scale="0.001 0.001 0.001"/>
       </geometry>
       <material name="${prefix}links_color"/>
@@ -173,23 +173,7 @@
   <link name="${prefix}ee_finger2">
     <visual>
-      <origin xyz="0 0 0" rpy="0 0 0"/>
-      <geometry>
-        <mesh filename="package://rover_arm_description/meshes/visual/end_effector_finger.stl" scale="0.001 0.001 0.001"/>
-      </geometry>
-      <material name="${prefix}links_color"/>
-    </visual>
-    <collision>
-      <origin xyz="0.016 ${0.14 / 2} ${- 0.022 / 2}" rpy="0 0 0"/>
-      <geometry>
-        <box size="0.042 0.14 0.022"/>
-      </geometry>
-    </collision>
-  </link>
-  <!-- finger 3 -->
-  <link name="${prefix}ee_finger3">
-    <visual>
-      <origin xyz="0 0 0" rpy="0 0 0"/>
-      <geometry>
-        <mesh filename="package://rover_arm_description/meshes/visual/end_effector_finger.stl" scale="0.001 0.001 0.001"/>
+      <origin xyz="0 0 0" rpy="${finger2_rotation_offset}"/>
+      <geometry>
+        <mesh filename="package://rover_arm_description/meshes/visual/two_finger_version/end_effector_finger.stl" scale="0.001 0.001 0.001"/>
       </geometry>
       <material name="${prefix}links_color"/>
@@ -278,6 +262,5 @@
     <child link="${prefix}ee_finger1"/>
     <origin xyz="${finger1_joint_pos}" rpy="${finger1_joint_rotation}"/>
-    <!-- Sliding Axis -->
-    <axis xyz="0 0 1"/>
+    <axis xyz="-1 0 0"/>
     <!-- Limits -->
     <limit lower="0.0" upper="${finger_rotation_upper_bound}" effort="50.0" velocity="1.0"/>
@@ -289,19 +272,9 @@
     <child link="${prefix}ee_finger2"/>
     <origin xyz="${finger2_joint_pos}" rpy="${finger2_joint_rotation}"/>
-    <axis xyz="0 0 1"/>
+    <axis xyz="1 0 0"/>
     <!-- Limits -->
     <limit lower="0.0" upper="${finger_rotation_upper_bound}" effort="50.0" velocity="1.0"/>
     <mimic joint="${prefix}slider_joint" multiplier="${relation_multip}" offset="0.0"/>
   </joint>
-  <!-- finger 3 joint-->
-  <joint name="${prefix}finger3_joint" type="revolute">
-    <parent link="${prefix}ee_base"/>
-    <child link="${prefix}ee_finger3"/>
-    <origin xyz="${finger3_joint_pos}" rpy="${finger3_joint_rotation}"/>
-    <axis xyz="0 0 1"/>
-    <!-- Limits -->
-    <limit lower="0.0" upper="${finger_rotation_upper_bound}" effort="50.0" velocity="1.0"/>
-    <mimic joint="${prefix}slider_joint" multiplier="${relation_multip}" offset="0.0"/>
-  </joint>
   </xacro:macro>
 </robot>
